Commit message: fix: GO2 urdf dae path error

File: resources/robots/go2/urdf/go2.urdf (robot description, URDF)
Before this commit: robot go2_description, 29 links, 28 joints
Links:
- link FL_calf: geometry collision cylinder length=0.05 radius=0.01; visual mesh filename=../meshes/calf.dae
- link FL_foot: geometry collision sphere radius=0.022; visual mesh filename=../meshes/foot.dae
- link FL_hip: geometry collision cylinder length=0.04 radius=0.046; visual mesh filename=../meshes/hip.dae
- link FL_thigh: geometry collision box size=0.16 0.0245 0.034; visual mesh filename=../meshes/thigh.dae
- link FR_calf: geometry collision cylinder length=0.05 radius=0.01; visual mesh filename=../meshes/calf_mirror.dae
- link FR_foot: geometry collision sphere radius=0.022; visual mesh filename=../meshes/foot.dae
- link FR_hip: geometry collision cylinder length=0.04 radius=0.046; visual mesh filename=../meshes/hip.dae
- link FR_thigh: geometry collision box size=0.16 0.0245 0.034; visual mesh filename=../meshes/thigh_mirror.dae
- link RL_calf: geometry collision cylinder length=0.05 radius=0.01; visual mesh filename=../meshes/calf.dae
- link RL_foot: geometry collision sphere radius=0.022; visual mesh filename=../meshes/foot.dae
- link RL_hip: geometry collision cylinder length=0.04 radius=0.046; visual mesh filename=../meshes/hip.dae
- link RL_thigh: geometry collision box size=0.16 0.0245 0.034; visual mesh filename=../meshes/thigh.dae
- link RR_calf: geometry collision cylinder length=0.05 radius=0.01; visual mesh filename=../meshes/calf_mirror.dae
- link RR_foot: geometry collision sphere radius=0.022; visual mesh filename=../meshes/foot.dae
- link RR_hip: geometry collision cylinder length=0.04 radius=0.046; visual mesh filename=../meshes/hip.dae
- link RR_thigh: geometry collision box size=0.16 0.0245 0.034; visual mesh filename=../meshes/thigh_mirror.dae
- link base: geometry collision box size=0.3762 0.0935 0.114; visual mesh filename=../meshes/base.dae

Commit message: commit: Go2 foot modification

File: resources/robots/go2/urdf/go2.urdf (robot description, URDF)
Before this commit: robot go2_description, 29 links, 28 joints
Links:
- removed link FL_calflower1
- removed link FR_calflower1
- removed link RL_calflower1
- removed link RR_calflower1
- added link FL_end; collision cylinder length=0.04 radius=0.01; visual cylinder length=0.04 radius=0.01
- added link FL_end1; collision cylinder length=0.04 radius=0.01; visual cylinder length=0.04 radius=0.01
- added link FL_end2; collision cylinder length=0.04 radius=0.01; visual cylinder length=0.04 radius=0.01
- added link FL_end3; collision cylinder length=0.02 radius=0.01; visual cylinder length=0.02 radius=0.01
- added link FL_foot1; collision sphere radius=0.015; visual sphere radius=0.015
- added link FR_end; collision cylinder length=0.04 radius=0.01; visual cylinder length=0.04 radius=0.01
- added link FR_end1; collision cylinder length=0.04 radius=0.01; visual cylinder length=0.04 radius=0.01
- added link FR_end2; collision cylinder length=0.04 radius=0.01; visual cylinder length=0.04 radius=0.01
- added link FR_end3; collision cylinder length=0.02 radius=0.01; visual cylinder length=0.02 radius=0.01
- added link FR_foot1; collision sphere radius=0.015; visual sphere radius=0.015
- added link RL_end; collision cylinder length=0.04 radius=0.01; visual cylinder length=0.04 radius=0.01
- added link RL_end1; collision cylinder length=0.04 radius=0.01; visual cylinder length=0.04 radius=0.01
- added link RL_end2; collision cylinder length=0.04 radius=0.01; visual cylinder length=0.04 radius=0.01
- added link RL_end3; collision cylinder length=0.02 radius=0.01; visual cylinder length=0.02 radius=0.01
- added link RL_foot1; collision sphere radius=0.015; visual sphere radius=0.015
- added link RR_end; collision cylinder length=0.04 radius=0.01; visual cylinder length=0.04 radius=0.01
- added link RR_end1; collision cylinder length=0.04 radius=0.01; visual cylinder length=0.04 radius=0.01
- added link RR_end2; collision cylinder length=0.04 radius=0.01; visual cylinder length=0.04 radius=0.01
- added link RR_end3; collision cylinder length=0.02 radius=0.01; visual cylinder length=0.02 radius=0.01
- added link RR_foot1; collision sphere radius=0.015; visual sphere radius=0.015
- link FL_calf: geometry collision cylinder length=0.05 radius=0.01; visual cylinder length=0.05 radius=0.01
- link FL_calflower: geometry collision cylinder length=0.08 radius=0.01; visual cylinder length=0.08 radius=0.01
- link FL_foot: mass 0.04 -> None; geometry collision sphere radius=0.02; visual sphere radius=0.02
- link FR_calf: geometry collision cylinder length=0.05 radius=0.01; visual cylinder length=0.05 radius=0.01
- link FR_calflower: geometry collision cylinder length=0.08 radius=0.01; visual cylinder length=0.08 radius=0.01
- link FR_foot: mass 0.04 -> None; geometry collision sphere radius=0.02; visual sphere radius=0.02
- link RL_calf: geometry collision cylinder length=0.05 radius=0.01; visual cylinder length=0.05 radius=0.01
- link RL_calflower: geometry collision cylinder length=0.08 radius=0.01; visual cylinder length=0.08 radius=0.01
- link RL_foot: mass 0.04 -> None; geometry collision sphere radius=0.02; visual sphere radius=0.02
- link RR_calf: geometry collision cylinder length=0.05 radius=0.01; visual cylinder length=0.05 radius=0.01
- link RR_calflower: geometry collision cylinder length=0.08 radius=0.01; visual cylinder length=0.08 radius=0.01
- link RR_foot: mass 0.04 -> None; geometry collision sphere radius=0.02; visual sphere radius=0.02
Joints:
- removed joint FL_calflower1_joint
- removed joint FR_calflower1_joint
- removed joint RL_calflower1_joint
- removed joint RR_calflower1_joint
- added joint FL_end1_joint: type fixed, parent FL_end, child FL_end1, origin xyz=-0.01 0 -0.03 rpy=0 0.8 0, axis 0 0 0
- added joint FL_end2_joint: type fixed, parent FL_calflower, child FL_end2, origin xyz=-0.01 0 -0.0 rpy=0 -0.8 0, axis 0 0 0
- added joint FL_end3_joint: type fixed, parent FL_end2, child FL_end3, origin xyz=-0.005 0 0.025 rpy=0 -0.4 0, axis 0 0 0
- added joint FL_end_joint: type fixed, parent FL_calflower, child FL_end, origin xyz=-0.01 0 -0.05 rpy=0 0.8 0, axis 0 0 0
- added joint FL_foot1_joint: type fixed, parent FL_end3, child FL_foot1, origin xyz=0 0 0.015 rpy=0 0 0, axis 0 0 0
- added joint FR_end1_joint: type fixed, parent FR_end, child FR_end1, origin xyz=-0.01 0 -0.03 rpy=0 0.8 0, axis 0 0 0
- added joint FR_end2_joint: type fixed, parent FR_calflower, child FR_end2, origin xyz=-0.01 0 -0.0 rpy=0 -0.8 0, axis 0 0 0
- added joint FR_end3_joint: type fixed, parent FR_end2, child FR_end3, origin xyz=-0.005 0 0.025 rpy=0 -0.4 0, axis 0 0 0
- added joint FR_end_joint: type fixed, parent FR_calflower, child FR_end, origin xyz=-0.01 0 -0.05 rpy=0 0.8 0, axis 0 0 0
- added joint FR_foot1_joint: type fixed, parent FR_end3, child FR_foot1, origin xyz=0 0 0.015 rpy=0 0 0, axis 0 0 0
- added joint RL_end1_joint: type fixed, parent RL_end, child RL_end1, origin xyz=-0.01 0 -0.03 rpy=0 0.8 0, axis 0 0 0
- added joint RL_end2_joint: type fixed, parent RL_calflower, child RL_end2, origin xyz=-0.01 0 -0.0 rpy=0 -0.8 0, axis 0 0 0
- added joint RL_end3_joint: type fixed, parent RL_end2, child RL_end3, origin xyz=-0.005 0 0.025 rpy=0 -0.4 0, axis 0 0 0
- added joint RL_end_joint: type fixed, parent RL_calflower, child RL_end, origin xyz=-0.01 0 -0.05 rpy=0 0.8 0, axis 0 0 0
- added joint RL_foot1_joint: type fixed, parent RL_end3, child RL_foot1, origin xyz=0 0 0.015 rpy=0 0 0, axis 0 0 0
- added joint RR_end1_joint: type fixed, parent RR_end, child RR_end1, origin xyz=-0.01 0 -0.03 rpy=0 0.8 0, axis 0 0 0
- added joint RR_end2_joint: type fixed, parent RR_calflower, child RR_end2, origin xyz=-0.01 0 -0.0 rpy=0 -0.8 0, axis 0 0 0
- added joint RR_end3_joint: type fixed, parent RR_end2, child RR_end3, origin xyz=-0.005 0 0.025 rpy=0 -0.4 0, axis 0 0 0
- added joint RR_end_joint: type fixed, parent RR_calflower, child RR_end, origin xyz=-0.01 0 -0.05 rpy=0 0.8 0, axis 0 0 0
- added joint RR_foot1_joint: type fixed, parent RR_end3, child RR_foot1, origin xyz=0 0 0.015 rpy=0 0 0, axis 0 0 0
- joint FL_calflower_joint: origin xyz=0.020 0 -0.148 rpy=0 0.05 0 -> xyz=0.018 0 -0.16 rpy=0 0.05 0
- joint FL_foot_joint: origin xyz=0 0 -0.213 rpy=0 0 0 -> xyz=0.005 0 -0.02 rpy=0 0 0; parent FL_calf -> FL_end1
- joint FR_calflower_joint: origin xyz=0.020 0 -0.148 rpy=0 0.05 0 -> xyz=0.018 0 -0.16 rpy=0 0.05 0
- joint FR_foot_joint: origin xyz=0 0 -0.213 rpy=0 0 0 -> xyz=0.005 0 -0.02 rpy=0 0 0; parent FR_calf -> FR_end1
- joint RL_calflower_joint: origin xyz=0.020 0 -0.148 rpy=0 0.05 0 -> xyz=0.018 0 -0.16 rpy=0 0.05 0
- joint RL_foot_joint: origin xyz=0 0 -0.213 rpy=0 0 0 -> xyz=0.005 0 -0.02 rpy=0 0 0; parent RL_calf -> RL_end1
- joint RR_calflower_joint: origin xyz=0.020 0 -0.148 rpy=0 0.05 0 -> xyz=0.018 0 -0.16 rpy=0 0.05 0
- joint RR_foot_joint: origin xyz=0 0 -0.213 rpy=0 0 0 -> xyz=0.005 0 -0.02 rpy=0 0 0; parent RR_calf -> RR_end1

Commit message: fix: invalid collision of foot

File: resources/robots/go2/urdf/go2.urdf (robot description, URDF)
Before this commit: robot go2_description, 45 links, 44 joints
Links:
- link FL_calf: geometry collision cylinder length=0.04 radius=0.01; visual cylinder length=0.04 radius=0.01
- link FL_calflower: geometry collision cylinder length=0.07 radius=0.01; visual cylinder length=0.07 radius=0.01
- link FL_end: geometry collision cylinder length=0.03 radius=0.01; visual cylinder length=0.03 radius=0.01
- link FL_end1: geometry collision cylinder length=0.03 radius=0.01; visual cylinder length=0.03 radius=0.01
- link FL_end2: geometry collision cylinder length=0.03 radius=0.01; visual cylinder length=0.03 radius=0.01
- link FL_end3: geometry collision cylinder length=0.01 radius=0.01; visual cylinder length=0.01 radius=0.01
- link FL_foot: mass None -> 0.014137; geometry collision sphere radius=0.015; visual sphere radius=0.015
- link FL_foot1: mass None -> 0.014137
- link FR_calf: geometry collision cylinder length=0.04 radius=0.01; visual cylinder length=0.04 radius=0.01
- link FR_calflower: geometry collision cylinder length=0.07 radius=0.01; visual cylinder length=0.07 radius=0.01
- link FR_end: geometry collision cylinder length=0.03 radius=0.01; visual cylinder length=0.03 radius=0.01
- link FR_end1: geometry collision cylinder length=0.03 radius=0.01; visual cylinder length=0.03 radius=0.01
- link FR_end2: geometry collision cylinder length=0.03 radius=0.01; visual cylinder length=0.03 radius=0.01
- link FR_end3: geometry collision cylinder length=0.01 radius=0.01; visual cylinder length=0.01 radius=0.01
- link FR_foot: mass None -> 0.014137; geometry collision sphere radius=0.015; visual sphere radius=0.015
- link FR_foot1: mass None -> 0.014137
- link RL_calf: geometry collision cylinder length=0.04 radius=0.01; visual cylinder length=0.04 radius=0.01
- link RL_calflower: geometry collision cylinder length=0.07 radius=0.01; visual cylinder length=0.07 radius=0.01
- link RL_end: geometry collision cylinder length=0.03 radius=0.01; visual cylinder length=0.03 radius=0.01
- link RL_end1: geometry collision cylinder length=0.03 radius=0.01; visual cylinder length=0.03 radius=0.01
- link RL_end2: geometry collision cylinder length=0.03 radius=0.01; visual cylinder length=0.03 radius=0.01
- link RL_end3: geometry collision cylinder length=0.01 radius=0.01; visual cylinder length=0.01 radius=0.01
- link RL_foot: mass None -> 0.014137; geometry collision sphere radius=0.015; visual sphere radius=0.015
- link RL_foot1: mass None -> 0.014137
- link RR_calf: geometry collision cylinder length=0.04 radius=0.01; visual cylinder length=0.04 radius=0.01
- link RR_calflower: geometry collision cylinder length=0.07 radius=0.01; visual cylinder length=0.07 radius=0.01
- link RR_end: geometry collision cylinder length=0.03 radius=0.01; visual cylinder length=0.03 radius=0.01
- link RR_end1: geometry collision cylinder length=0.03 radius=0.01; visual cylinder length=0.03 radius=0.01
- link RR_end2: geometry collision cylinder length=0.03 radius=0.01; visual cylinder length=0.03 radius=0.01
- link RR_end3: geometry collision cylinder length=0.01 radius=0.01; visual cylinder length=0.01 radius=0.01
- link RR_foot: mass None -> 0.014137; geometry collision sphere radius=0.015; visual sphere radius=0.015
- link RR_foot1: mass None -> 0.014137
Joints:
- joint FL_foot_joint: origin xyz=0.005 0 -0.02 rpy=0 0 0 -> xyz=0.002 0 -0.02 rpy=0 0 0
- joint FR_foot_joint: origin xyz=0.005 0 -0.02 rpy=0 0 0 -> xyz=0.002 0 -0.02 rpy=0 0 0
- joint RL_foot_joint: origin xyz=0.005 0 -0.02 rpy=0 0 0 -> xyz=0.002 0 -0.02 rpy=0 0 0
- joint RR_foot_joint: origin xyz=0.005 0 -0.02 rpy=0 0 0 -> xyz=0.002 0 -0.02 rpy=0 0 0

Commit message: update: Go2 end effector

File: resources/robots/go2/urdf/go2.urdf (robot description, URDF)
Before this commit: robot go2_description, 45 links, 44 joints
Links:
- removed link FL_end3
- removed link FR_end3
- removed link RL_end1
- removed link RR_end1
Joints:
- removed joint FL_end3_joint
- removed joint FR_end3_joint
- removed joint RL_end1_joint
- removed joint RR_end1_joint
- joint FL_foot1_joint: origin xyz=0 0 0.015 rpy=0 0 0 -> xyz=0 0 0.02 rpy=0 0 0; parent FL_end3 -> FL_end2
- joint FR_foot1_joint: origin xyz=0 0 0.015 rpy=0 0 0 -> xyz=0 0 0.02 rpy=0 0 0; parent FR_end3 -> FR_end2
- joint RL_foot_joint: parent RL_end1 -> RL_end
- joint RR_foot_joint: parent RR_end1 -> RR_end

Commit message: update: decouple calf and effector and recalc

File: resources/robots/go2/urdf/go2.urdf (robot description, URDF)
Before this commit: robot go2_description, 41 links, 40 joints
Links:
- added link FL_effector, mass 0.025446900494077326; collision cylinder length=0.03 radius=0.01; visual cylinder length=0.03 radius=0.01
- added link FR_effector, mass 0.025446900494077326; collision cylinder length=0.03 radius=0.01; visual cylinder length=0.03 radius=0.01
- added link RL_effector, mass 0.025446900494077326; collision cylinder length=0.03 radius=0.01; visual cylinder length=0.03 radius=0.01
- added link RR_effector, mass 0.025446900494077326; collision cylinder length=0.03 radius=0.01; visual cylinder length=0.03 radius=0.01
- link FL_calf: mass 0.154 -> 0.08482300164692443; geometry collision cylinder length=0.04 radius=0.01; visual cylinder length=0.1 radius=0.01
- link FL_calflower: mass None -> 0.03392920065876977; geometry collision cylinder length=0.04 radius=0.01; visual cylinder length=0.04 radius=0.01
- link FL_end: mass None -> 0.025446900494077326
- link FL_end1: mass None -> 0.025446900494077326
- link FL_end2: mass None -> 0.025446900494077326
- link FL_foot: mass 0.014137 -> 0.03817035074111598
- link FL_foot1: mass 0.014137 -> 0.03817035074111598
- link FR_calf: mass 0.154 -> 0.08482300164692443; geometry collision cylinder length=0.04 radius=0.01; visual cylinder length=0.1 radius=0.01
- link FR_calflower: mass None -> 0.03392920065876977; geometry collision cylinder length=0.04 radius=0.01; visual cylinder length=0.04 radius=0.01
- link FR_end: mass None -> 0.025446900494077326
- link FR_end1: mass None -> 0.025446900494077326
- link FR_end2: mass None -> 0.025446900494077326
- link FR_foot: mass 0.014137 -> 0.03817035074111598
- link FR_foot1: mass 0.014137 -> 0.03817035074111598
- link RL_calf: mass 0.154 -> 0.08482300164692443; geometry collision cylinder length=0.04 radius=0.01; visual cylinder length=0.1 radius=0.01
- link RL_calflower: mass None -> 0.03392920065876977; geometry collision cylinder length=0.04 radius=0.01; visual cylinder length=0.04 radius=0.01
- link RL_end: mass None -> 0.025446900494077326
- link RL_end2: mass None -> 0.025446900494077326
- link RL_end3: mass None -> 0.025446900494077326; geometry collision cylinder length=0.03 radius=0.01; visual cylinder length=0.03 radius=0.01
- link RL_foot: mass 0.014137 -> 0.03817035074111598
- link RL_foot1: mass 0.014137 -> 0.03817035074111598
- link RR_calf: mass 0.154 -> 0.08482300164692443; geometry collision cylinder length=0.04 radius=0.01; visual cylinder length=0.1 radius=0.01
- link RR_calflower: mass None -> 0.03392920065876977; geometry collision cylinder length=0.04 radius=0.01; visual cylinder length=0.04 radius=0.01
- link RR_end: mass None -> 0.025446900494077326
- link RR_end2: mass None -> 0.025446900494077326
- link RR_end3: mass None -> 0.025446900494077326; geometry collision cylinder length=0.03 radius=0.01; visual cylinder length=0.03 radius=0.01
- link RR_foot: mass 0.014137 -> 0.03817035074111598
- link RR_foot1: mass 0.014137 -> 0.03817035074111598
Joints:
- added joint FL_effector_joint: type fixed, parent FL_calflower, child FL_effector, origin xyz=0 0 -0.04 rpy=0 0 0, axis 0 0 0
- added joint FR_effector_joint: type fixed, parent FR_calflower, child FR_effector, origin xyz=0 0 -0.04 rpy=0 0 0, axis 0 0 0
- added joint RL_effector_joint: type fixed, parent RL_calflower, child RL_effector, origin xyz=0 0 -0.04 rpy=0 0 0, axis 0 0 0
- added joint RR_effector_joint: type fixed, parent RR_calflower, child RR_effector, origin xyz=0 0 -0.04 rpy=0 0 0, axis 0 0 0
- joint FL_calflower_joint: origin xyz=0.018 0 -0.16 rpy=0 0.05 0 -> xyz=0.018 0 -0.14 rpy=0 0.05 0
- joint FL_end1_joint: origin xyz=-0.01 0 -0.03 rpy=0 0.8 0 -> xyz=-0.012 0 -0.03 rpy=0 0.785 0
- joint FL_end2_joint: origin xyz=-0.01 0 -0.0 rpy=0 -0.8 0 -> xyz=-0.012 0 0.03 rpy=0 -0.785 0; parent FL_calflower -> FL_effector
- joint FL_end_joint: origin xyz=-0.01 0 -0.05 rpy=0 0.8 0 -> xyz=-0.012 0 -0.03 rpy=0 0.785 0; parent FL_calflower -> FL_effector
- joint FL_foot_joint: origin xyz=0.002 0 -0.02 rpy=0 0 0 -> xyz=0 0 -0.02 rpy=0 0 0
- joint FR_calflower_joint: origin xyz=0.018 0 -0.16 rpy=0 0.05 0 -> xyz=0.018 0 -0.14 rpy=0 0.05 0
- joint FR_end1_joint: origin xyz=-0.01 0 -0.03 rpy=0 0.8 0 -> xyz=-0.012 0 -0.03 rpy=0 0.785 0
- joint FR_end2_joint: origin xyz=-0.01 0 -0.0 rpy=0 -0.8 0 -> xyz=-0.012 0 0.03 rpy=0 -0.785 0; parent FR_calflower -> FR_effector
- joint FR_end_joint: origin xyz=-0.01 0 -0.05 rpy=0 0.8 0 -> xyz=-0.012 0 -0.03 rpy=0 0.785 0; parent FR_calflower -> FR_effector
- joint FR_foot_joint: origin xyz=0.002 0 -0.02 rpy=0 0 0 -> xyz=0 0 -0.02 rpy=0 0 0
- joint RL_calflower_joint: origin xyz=0.018 0 -0.16 rpy=0 0.05 0 -> xyz=0.018 0 -0.14 rpy=0 0.05 0
- joint RL_end2_joint: origin xyz=-0.01 0 -0.0 rpy=0 -0.8 0 -> xyz=-0.012 0 0.03 rpy=0 -0.785 0; parent RL_calflower -> RL_effector
- joint RL_end3_joint: origin xyz=-0.005 0 0.025 rpy=0 -0.4 0 -> xyz=-0.012 0 0.03 rpy=0 -0.785 0
- joint RL_end_joint: origin xyz=-0.01 0 -0.05 rpy=0 0.8 0 -> xyz=-0.012 0 -0.03 rpy=0 0.785 0; parent RL_calflower -> RL_effector
- joint RL_foot1_joint: origin xyz=0 0 0.015 rpy=0 0 0 -> xyz=0 0 0.02 rpy=0 0 0
- joint RL_foot_joint: origin xyz=0.002 0 -0.02 rpy=0 0 0 -> xyz=0 0 -0.02 rpy=0 0 0
- joint RR_calflower_joint: origin xyz=0.018 0 -0.16 rpy=0 0.05 0 -> xyz=0.018 0 -0.14 rpy=0 0.05 0
- joint RR_end2_joint: origin xyz=-0.01 0 -0.0 rpy=0 -0.8 0 -> xyz=-0.012 0 0.03 rpy=0 -0.785 0; parent RR_calflower -> RR_effector
- joint RR_end3_joint: origin xyz=-0.005 0 0.025 rpy=0 -0.4 0 -> xyz=-0.012 0 0.03 rpy=0 -0.785 0
- joint RR_end_joint: origin xyz=-0.01 0 -0.05 rpy=0 0.8 0 -> xyz=-0.012 0 -0.03 rpy=0 0.785 0; parent RR_calflower -> RR_effector
- joint RR_foot1_joint: origin xyz=0 0 0.015 rpy=0 0 0 -> xyz=0 0 0.02 rpy=0 0 0
- joint RR_foot_joint: origin xyz=0.002 0 -0.02 rpy=0 0 0 -> xyz=0 0 -0.02 rpy=0 0 0
