Commit message: update: adapt urdf to actual end effector

File: resources/robots/go2/urdf/go2.urdf (robot description, URDF)
Before this commit: robot go2_description, 45 links, 44 joints
Links:
- link FL_calf: mass 0.08482300164692443 -> 0.154; geometry collision cylinder length=0.04 radius=0.01; visual mesh filename=../meshes/calf.dae
- link FL_calflower: mass 0.03392920065876977 -> None; geometry collision cylinder length=0.1 radius=0.01
- link FL_effector: mass 0.025446900494077326 -> 0.011686724671354032
- link FL_end: mass 0.025446900494077326 -> 0.011686724671354032
- link FL_end1: mass 0.025446900494077326 -> 0.011686724671354032
- link FL_end2: mass 0.025446900494077326 -> 0.011686724671354032
- link FL_foot: mass 0.03817035074111598 -> 0.016257741982327174
- link FL_foot1: mass 0.03817035074111598 -> 0.016257741982327174
- link FR_calf: mass 0.08482300164692443 -> 0.154; geometry collision cylinder length=0.04 radius=0.01; visual mesh filename=../meshes/calf_mirror.dae
- link FR_calflower: mass 0.03392920065876977 -> None; geometry collision cylinder length=0.1 radius=0.01
- link FR_effector: mass 0.025446900494077326 -> 0.011686724671354032
- link FR_end: mass 0.025446900494077326 -> 0.011686724671354032
- link FR_end1: mass 0.025446900494077326 -> 0.011686724671354032
- link FR_end2: mass 0.025446900494077326 -> 0.011686724671354032
- link FR_foot: mass 0.03817035074111598 -> 0.016257741982327174
- link FR_foot1: mass 0.03817035074111598 -> 0.016257741982327174
- link RL_calf: mass 0.08482300164692443 -> 0.154; geometry collision cylinder length=0.04 radius=0.01; visual mesh filename=../meshes/calf.dae
- link RL_calflower: mass 0.03392920065876977 -> None; geometry collision cylinder length=0.1 radius=0.01
- link RL_effector: mass 0.025446900494077326 -> 0.011686724671354032
- link RL_end: mass 0.025446900494077326 -> 0.011686724671354032
- link RL_end2: mass 0.025446900494077326 -> 0.011686724671354032
- link RL_end3: mass 0.025446900494077326 -> 0.011686724671354032
- link RL_foot: mass 0.03817035074111598 -> 0.016257741982327174
- link RL_foot1: mass 0.03817035074111598 -> 0.016257741982327174
- link RR_calf: mass 0.08482300164692443 -> 0.154; geometry collision cylinder length=0.04 radius=0.01; visual mesh filename=../meshes/calf_mirror.dae
- link RR_calflower: mass 0.03392920065876977 -> None; geometry collision cylinder length=0.1 radius=0.01
- link RR_effector: mass 0.025446900494077326 -> 0.011686724671354032
- link RR_end: mass 0.025446900494077326 -> 0.011686724671354032
- link RR_end2: mass 0.025446900494077326 -> 0.011686724671354032
- link RR_end3: mass 0.025446900494077326 -> 0.011686724671354032
- link RR_foot: mass 0.03817035074111598 -> 0.016257741982327174
- link RR_foot1: mass 0.03817035074111598 -> 0.016257741982327174
Joints:
- joint FL_effector_joint: origin xyz=0 0 -0.04 rpy=0 0 0 -> xyz=-0.03 0 -0.04 rpy=0 0.1 0
- joint FL_foot1_joint: origin xyz=0 0 0.02 rpy=0 0 0 -> xyz=0 0 0.015 rpy=0 0 0
- joint FL_foot_joint: origin xyz=0 0 -0.02 rpy=0 0 0 -> xyz=0 0 -0.015 rpy=0 0 0
- joint FR_effector_joint: origin xyz=0 0 -0.04 rpy=0 0 0 -> xyz=-0.03 0 -0.04 rpy=0 0.1 0
- joint FR_foot1_joint: origin xyz=0 0 0.02 rpy=0 0 0 -> xyz=0 0 0.015 rpy=0 0 0
- joint FR_foot_joint: origin xyz=0 0 -0.02 rpy=0 0 0 -> xyz=0 0 -0.015 rpy=0 0 0
- joint RL_effector_joint: origin xyz=0 0 -0.04 rpy=0 0 0 -> xyz=-0.03 0 -0.04 rpy=0 0.1 0
- joint RL_foot1_joint: origin xyz=0 0 0.02 rpy=0 0 0 -> xyz=0 0 0.015 rpy=0 0 0
- joint RL_foot_joint: origin xyz=0 0 -0.02 rpy=0 0 0 -> xyz=0 0 -0.015 rpy=0 0 0
- joint RR_effector_joint: origin xyz=0 0 -0.04 rpy=0 0 0 -> xyz=-0.03 0 -0.04 rpy=0 0.1 0
- joint RR_foot1_joint: origin xyz=0 0 0.02 rpy=0 0 0 -> xyz=0 0 0.015 rpy=0 0 0
- joint RR_foot_joint: origin xyz=0 0 -0.02 rpy=0 0 0 -> xyz=0 0 -0.015 rpy=0 0 0
