Commit message: update: simulate deformation damping

File: resources/robots/go2/urdf/go2.urdf (robot description, URDF)
Before this commit: robot go2_description, 57 links, 56 joints
Links:
- removed link FL_foot
- removed link FL_foot1
- removed link FR_foot
- removed link FR_foot1
- removed link RL_foot
- removed link RL_foot1
- removed link RR_foot
- removed link RR_foot1
- added link FL_foot_front, mass 0.016257741982327174; collision sphere radius=0.015; visual sphere radius=0.015
- added link FL_foot_rear, mass 0.016257741982327174; collision sphere radius=0.015; visual sphere radius=0.015
- added link FR_foot_front, mass 0.016257741982327174; collision sphere radius=0.015; visual sphere radius=0.015
- added link FR_foot_rear, mass 0.016257741982327174; collision sphere radius=0.015; visual sphere radius=0.015
- added link RL_foot_front, mass 0.016257741982327174; collision sphere radius=0.015; visual sphere radius=0.015
- added link RL_foot_rear, mass 0.016257741982327174; collision sphere radius=0.015; visual sphere radius=0.015
- added link RR_foot_front, mass 0.016257741982327174; collision sphere radius=0.015; visual sphere radius=0.015
- added link RR_foot_rear, mass 0.016257741982327174; collision sphere radius=0.015; visual sphere radius=0.015
Joints:
- removed joint FL_foot1_joint
- removed joint FL_foot_joint
- removed joint FR_foot1_joint
- removed joint FR_foot_joint
- removed joint RL_foot1_joint
- removed joint RL_foot_joint
- removed joint RR_foot1_joint
- removed joint RR_foot_joint
- added joint FL_foot_front_joint: type fixed, parent FL_end1, child FL_foot_front, origin xyz=0 0 -0.015 rpy=0 0 0, axis 0 0 0
- added joint FL_foot_rear_joint: type fixed, parent FL_end2, child FL_foot_rear, origin xyz=0 0 0.015 rpy=0 0 0, axis 0 0 0
- added joint FR_foot_front_joint: type fixed, parent FR_end1, child FR_foot_front, origin xyz=0 0 -0.015 rpy=0 0 0, axis 0 0 0
- added joint FR_foot_rear_joint: type fixed, parent FR_end2, child FR_foot_rear, origin xyz=0 0 0.015 rpy=0 0 0, axis 0 0 0
- added joint RL_foot_front_joint: type fixed, parent RL_end, child RL_foot_front, origin xyz=0 0 -0.015 rpy=0 0 0, axis 0 0 0
- added joint RL_foot_rear_joint: type fixed, parent RL_end3, child RL_foot_rear, origin xyz=0 0 0.015 rpy=0 0 0, axis 0 0 0
- added joint RR_foot_front_joint: type fixed, parent RR_end, child RR_foot_front, origin xyz=0 0 -0.015 rpy=0 0 0, axis 0 0 0
- added joint RR_foot_rear_joint: type fixed, parent RR_end3, child RR_foot_rear, origin xyz=0 0 0.015 rpy=0 0 0, axis 0 0 0

Commit message: update: Go2 urdf according to real effector

File: resources/robots/go2/urdf/go2.urdf (robot description, URDF)
Before this commit: robot go2_description, 57 links, 56 joints
Links:
- link FL_effector: mass 0.011686724671354032 -> 0.01413716694115407
- link FL_end: mass 0.011686724671354032 -> 0.01413716694115407
- link FL_end1: mass 0.011686724671354032 -> 0.01413716694115407
- link FL_end2: mass 0.011686724671354032 -> 0.01413716694115407
- link FL_foot_front: mass 0.016257741982327174 -> 0.0212057504117311
- link FL_foot_rear: mass 0.016257741982327174 -> 0.0212057504117311
- link FR_effector: mass 0.011686724671354032 -> 0.01413716694115407
- link FR_end: mass 0.011686724671354032 -> 0.01413716694115407
- link FR_end1: mass 0.011686724671354032 -> 0.01413716694115407
- link FR_end2: mass 0.011686724671354032 -> 0.01413716694115407
- link FR_foot_front: mass 0.016257741982327174 -> 0.0212057504117311
- link FR_foot_rear: mass 0.016257741982327174 -> 0.0212057504117311
- link RL_effector: mass 0.011686724671354032 -> 0.01413716694115407
- link RL_end: mass 0.011686724671354032 -> 0.01413716694115407
- link RL_end2: mass 0.011686724671354032 -> 0.01413716694115407
- link RL_end3: mass 0.011686724671354032 -> 0.01413716694115407
- link RL_foot_front: mass 0.016257741982327174 -> 0.0212057504117311
- link RL_foot_rear: mass 0.016257741982327174 -> 0.0212057504117311
- link RR_effector: mass 0.011686724671354032 -> 0.01413716694115407
- link RR_end: mass 0.011686724671354032 -> 0.01413716694115407
- link RR_end2: mass 0.011686724671354032 -> 0.01413716694115407
- link RR_end3: mass 0.011686724671354032 -> 0.01413716694115407
- link RR_foot_front: mass 0.016257741982327174 -> 0.0212057504117311
- link RR_foot_rear: mass 0.016257741982327174 -> 0.0212057504117311
Joints:
- joint FL_effector_joint: origin xyz=-0.03 0 -0.04 rpy=0 0.1 0 -> xyz=-0.03 0 -0.042 rpy=0 0.12 0
- joint FL_foot_front_joint: origin xyz=0 0 -0.015 rpy=0 0 0 -> xyz=-0.003 0 -0.023 rpy=0 0 0
- joint FL_foot_rear_joint: origin xyz=0 0 0.015 rpy=0 0 0 -> xyz=-0.003 0 0.023 rpy=0 0 0
- joint FR_effector_joint: origin xyz=-0.03 0 -0.04 rpy=0 0.1 0 -> xyz=-0.03 0 -0.042 rpy=0 0.12 0
- joint FR_foot_front_joint: origin xyz=0 0 -0.015 rpy=0 0 0 -> xyz=-0.003 0 -0.023 rpy=0 0 0
- joint FR_foot_rear_joint: origin xyz=0 0 0.015 rpy=0 0 0 -> xyz=-0.003 0 0.023 rpy=0 0 0
- joint RL_effector_joint: origin xyz=-0.03 0 -0.04 rpy=0 0.1 0 -> xyz=-0.03 0 -0.042 rpy=0 0.12 0
- joint RL_foot_front_joint: origin xyz=0 0 -0.015 rpy=0 0 0 -> xyz=-0.003 0 -0.023 rpy=0 0 0
- joint RL_foot_rear_joint: origin xyz=0 0 0.015 rpy=0 0 0 -> xyz=-0.003 0 0.023 rpy=0 0 0
- joint RR_effector_joint: origin xyz=-0.03 0 -0.04 rpy=0 0.1 0 -> xyz=-0.03 0 -0.042 rpy=0 0.12 0
- joint RR_foot_front_joint: origin xyz=0 0 -0.015 rpy=0 0 0 -> xyz=-0.003 0 -0.023 rpy=0 0 0
- joint RR_foot_rear_joint: origin xyz=0 0 0.015 rpy=0 0 0 -> xyz=-0.003 0 0.023 rpy=0 0 0

Commit message: update: urdf according to solidworks model

File: resources/robots/go2/urdf/go2.urdf (robot description, URDF)
Before this commit: robot go2_description, 57 links, 56 joints
Links:
- link FL_effector: mass 0.01413716694115407 -> 0.120
- link FL_end: mass 0.01413716694115407 -> None
- link FL_end1: mass 0.01413716694115407 -> None
- link FL_end2: mass 0.01413716694115407 -> None
- link FR_effector: mass 0.01413716694115407 -> 0.120
- link FR_end: mass 0.01413716694115407 -> None
- link FR_end1: mass 0.01413716694115407 -> None
- link FR_end2: mass 0.01413716694115407 -> None
- link RL_effector: mass 0.01413716694115407 -> 0.120
- link RL_end: mass 0.01413716694115407 -> None
- link RL_end2: mass 0.01413716694115407 -> None
- link RL_end3: mass 0.01413716694115407 -> None
- link RR_effector: mass 0.01413716694115407 -> 0.120
- link RR_end: mass 0.01413716694115407 -> None
- link RR_end2: mass 0.01413716694115407 -> None
- link RR_end3: mass 0.01413716694115407 -> None

Commit message: fix: urdf missing foot

File: resources/robots/go2/urdf/go2.urdf (robot description, URDF)
Before this commit: robot go2_description, 57 links, 56 joints
Links:
- added link FL_foot, mass 0.04; collision sphere radius=0.022; visual mesh filename=../dae/foot.dae
- added link FR_foot, mass 0.04; collision sphere radius=0.022; visual mesh filename=../dae/foot.dae
- added link RL_foot, mass 0.04; collision sphere radius=0.022; visual mesh filename=../dae/foot.dae
- added link RR_foot, mass 0.04; collision sphere radius=0.022; visual mesh filename=../dae/foot.dae
Joints:
- added joint FL_foot_joint: type fixed, parent FL_calf, child FL_foot, origin xyz=0 0 -0.213 rpy=0 0 0, axis 0 0 0
- added joint FR_foot_joint: type fixed, parent FR_calf, child FR_foot, origin xyz=0 0 -0.213 rpy=0 0 0, axis 0 0 0
- added joint RL_foot_joint: type fixed, parent RL_calf, child RL_foot, origin xyz=0 0 -0.213 rpy=0 0 0, axis 0 0 0
- added joint RR_foot_joint: type fixed, parent RR_calf, child RR_foot, origin xyz=0 0 -0.213 rpy=0 0 0, axis 0 0 0

Commit message: fix: missing foot dae

File: resources/robots/go2/urdf/go2.urdf (robot description, URDF)
Before this commit: robot go2_description, 61 links, 60 joints
Links:
- link FL_foot: geometry collision sphere radius=0.022
- link FR_foot: geometry collision sphere radius=0.022
- link RL_foot: geometry collision sphere radius=0.022
- link RR_foot: geometry collision sphere radius=0.022

Commit message: update: add effector center link to calc dist

File: resources/robots/go2/urdf/go2.urdf (robot description, URDF)
Before this commit: robot go2_description, 61 links, 60 joints
Links:
- added link FL_effector_center
- added link FR_effector_center
- added link RL_effector_center
- added link RR_effector_center
Joints:
- added joint FL_effector_center_joint: type fixed, parent FL_effector, child FL_effector_center, origin xyz=-0.04 0 0 rpy=0 0 0, axis 0 0 0
- added joint FR_effector_center_joint: type fixed, parent FR_effector, child FR_effector_center, origin xyz=-0.04 0 0 rpy=0 0 0, axis 0 0 0
- added joint RL_effector_center_joint: type fixed, parent RL_effector, child RL_effector_center, origin xyz=-0.04 0 0 rpy=0 0 0, axis 0 0 0
- added joint RR_effector_center_joint: type fixed, parent RR_effector, child RR_effector_center, origin xyz=-0.04 0 0 rpy=0 0 0, axis 0 0 0

Commit message: update: increase base link thickness to avoid deploy collision

File: resources/robots/go2/urdf/go2.urdf (robot description, URDF)
Before this commit: robot go2_description, 65 links, 64 joints
Links:
- link base: geometry collision box size=0.3762 0.07 0.18; visual mesh filename=../meshes/base.dae
